Commit message: completed kf description - bad buoyancy still

File: kingfisher_description/urdf/base.urdf.xacro (robot description, xacro)
@@ -44,5 +44,5 @@
     <!-- PROPERTY LIST -->
     <!--All units in m-kg-s-radians unit system -->
-    <property name="M_PI" value="3.1415926535897931" />
+    <xacro:property name="M_PI" value="3.1415926535897931" />
     <!-- BASE-FOOTPRINT -->
     <!-- base_footprint is a fictitious link(frame) that is on the ground right below base_link origin, navigation stack depends on this frame -->
@@ -51,7 +51,5 @@
             <mass value="0.0001" />
             <origin xyz="0 0 0" />
-            <inertia ixx="0.0001" ixy="0.0" ixz="0.0"
-                iyy="0.0001" iyz="0.0"
-                izz="0.0001" />
+            <inertia ixx="0.0001" ixy="0.0" ixz="0.0" iyy="0.0001" iyz="0.0" izz="0.0001" />
         </inertial>
         <visual>
@@ -66,5 +64,5 @@
     </gazebo>
     <joint name="base_footprint_joint" type="fixed">
-    <origin xyz="0 0 0" rpy="0 0 0" />
+        <origin xyz="0 0 0" rpy="0 0 0" />
         <parent link="base_footprint"/>
         <child link="base_link" />
@@ -88,9 +86,39 @@
         </visual>
         <collision>
-          <origin xyz="0 0 0" rpy="0 0 0" />
-          <geometry>
-                <box size = "0.1 0.1 0.1"/> <!--making it slightly bigger in x and z direction-->
+            <origin xyz="0 0 0" rpy="0 0 0" />
+            <geometry>
+                <box size = "0.1 0.1 0.1"/>
+                <!--making it slightly bigger in x and z direction-->
             </geometry>
         </collision>
+    </link>
+    <xacro:property name="camera_link" value="0.05" />
+    <!-- Size of square 'camera' box -->
+    <joint name="camera_joint" type="fixed">
+        <axis xyz="0 1 0" />
+        <origin xyz="${camera_link} 0 1" rpy="0 0 0"/>
+        <parent link="base_link"/>
+        <child link="camera_link"/>
+    </joint>
+    <!-- Camera -->
+    <link name="camera_link">
+        <collision>
+            <origin xyz="0 0 0" rpy="0 0 0"/>
+            <geometry>
+                <box size="${camera_link} ${camera_link} ${camera_link}"/>
+            </geometry>
+        </collision>
+        <visual>
+            <origin xyz="0 0 0" rpy="0 0 0"/>
+            <geometry>
+                <box size="${camera_link} ${camera_link} ${camera_link}"/>
+            </geometry>
+            <material name="red"/>
+        </visual>
+        <inertial>
+            <mass value="1e-5" />
+            <origin xyz="0 0 0" rpy="0 0 0"/>
+            <inertia ixx="1e-6" ixy="0" ixz="0" iyy="1e-6" iyz="0" izz="1e-6" />
+        </inertial>
     </link>
     <gazebo reference="base_link">
@@ -100,29 +128,13 @@
     <!-- PANEL-LINKS -->
     <!-- Top Plate -->
-    <kingfisher_part parent="base_footprint" name="left_panel" mesh="left_panel"
-          translateX="0.0" translateY="-0.35" translateZ="0.05"
-          rotateX="${M_PI/2}" rotateY="0.0" rotateZ="${M_PI/2}"
-          color="Yellow" />
+    <kingfisher_part parent="base_footprint" name="left_panel" mesh="left_panel" translateX="0.0" translateY="-0.35" translateZ="0.05" rotateX="${M_PI/2}" rotateY="0.0" rotateZ="${M_PI/2}" color="Yellow" />
     <gazebo reference="base_footprint_left_panel_part">
         <material>Gazebo/Yellow</material>
     </gazebo>
-    <kingfisher_part parent="base_footprint" name="right_panel" mesh="right_panel"
-          translateX="0.0" translateY="0.35" translateZ="0.05"
-          rotateX="${M_PI/2}" rotateY="0.0" rotateZ="${-M_PI/2}"
-          color="Yellow" />
+    <kingfisher_part parent="base_footprint" name="right_panel" mesh="right_panel" translateX="0.0" translateY="0.35" translateZ="0.05" rotateX="${M_PI/2}" rotateY="0.0" rotateZ="${-M_PI/2}" color="Yellow" />
     <gazebo reference="base_footprint_right_panel_part">
         <material>Gazebo/Yellow</material>
     </gazebo>
     <!--Gazebo Plugin for simulating Kingfisher dynamics-->
-    <gazebo>
-      <plugin name="kingfisher_dynamic" filename="libkingfisher_gazebo_plugins.so">
-            <maxForce>62.0</maxForce>
-            <bodyName>base_link</bodyName>
-            <waterDensity>997.7735</waterDensity>
-            <waterLevel>1</waterLevel>
-            <xyzDampingFactor>20.0</xyzDampingFactor>
-            <yawDampingFactor>20.0</yawDampingFactor>
-            <rolPitDampingFactor>5.0</rolPitDampingFactor>
-        </plugin>
-    </gazebo>
+    <!-- <gazebo><plugin name="kingfisher_dynamic" filename="libkingfisher_gazebo_plugins.so"><maxForce>62.0</maxForce><bodyName>base_link</bodyName><waterDensity>997.7735</waterDensity><waterLevel>5</waterLevel><xyzDampingFactor>20.0</xyzDampingFactor><yawDampingFactor>20.0</yawDampingFactor><rolPitDampingFactor>5.0</rolPitDampingFactor></plugin></gazebo> -->
 </robot>

File: kingfisher_description/urdf/kingfisher_robotx.xacro (robot description, xacro)
@@ -1,10 +1,28 @@
 <?xml version="1.0"?>
-<robot name="kingfisher"
-    xmlns:sensor="http://playerstage.sourceforge.net/gazebo/xmlschema/#sensor"
-    xmlns:controller="http://playerstage.sourceforge.net/gazebo/xmlschema/#controller"
-    xmlns:interface="http://playerstage.sourceforge.net/gazebo/xmlschema/#interface"
-    xmlns:xacro="http://ros.org/wiki/xacro">
-    <!-- Included URDF Files -->
-    <arg name="sonar_enabled" default="false"/>
-    <xacro:include filename="$(find kingfisher_description)/urdf/standard.urdf.xacro" />
+<robot
+  xmlns:xacro="http://ros.org/wiki/xacro" name="Kingfisher">
+  <!-- Included URDF Files -->
+  <xacro:arg name="sonar_enabled" default="false"/>
+  <xacro:include filename="$(find kingfisher_description)/urdf/standard.urdf.xacro" />
+  <!-- Attach hydrodynamics plugin -->
+  <xacro:include filename="$(find robotx_gazebo)/urdf/kingfisher_gazebo_dynamics_plugin.xacro" />
+  <xacro:usv_dynamics_gazebo name="kingfisher_dynamics_plugin"/>
+  <!-- Attach wind plugin -->
+  <xacro:include filename="$(find robotx_gazebo)/urdf/kingfisher_gazebo_wind_plugin.xacro" />
+  <xacro:usv_wind_gazebo name="kingfisher_wind_plugin"/>
+  <!-- Attach thrust plugin -->
+  <xacro:include filename="$(find robotx_gazebo)/urdf/kingfisher_gazebo_thrust_plugin.xacro" />
+  <xacro:usv_thrust_gazebo name="kingfisher_thrust_plugin"/>
+  <!-- Attach Camera plugin -->
+  <xacro:include filename="$(find kingfisher_description)/urdf/sensor_camera.xacro" />
+  <xacro:kingfisher_gazebo_camera name="kingfisher_camera1"/>
+  <!-- Attach IMU plugin -->
+  <xacro:include filename="$(find kingfisher_description)/urdf/sensor_imu.xacro" />
+  <xacro:kingfisher_gazebo_imu name="kingfisher_imu"/>
+  <!-- Attach GPS plugin -->
+  <xacro:include filename="$(find kingfisher_description)/urdf/sensor_gps.xacro" />
+  <xacro:kingfisher_gazebo_gps name="kingfisher_gps"/>
+  <!-- Attach P3D plugin -->
+  <xacro:include filename="$(find kingfisher_description)/urdf/sensor_p3d.xacro" />
+  <xacro:kingfisher_gazebo_p3d name="kingfisher_p3d"/>
 </robot>

File: kingfisher_description/urdf/parts.urdf.xacro (robot description, xacro)
@@ -32,17 +32,17 @@
 	xmlns:interface="http://playerstage.sourceforge.net/gazebo/xmlschema/#interface"
 	xmlns:xacro="http://ros.org/wiki/xacro" name="kingfisher_part">
-	<property name="x_com" value="0.00000000" /> <!-- com : center of mass -->
-	<property name="y_com" value="0.00000000" /> <!-- com : center of mass -->
-	<property name="z_com" value="0.00000000" /> <!-- com : center of mass -->
-	<property name="x_size" value="1.0" />
-	<property name="y_size" value="1.0" />
-	<property name="z_size" value="1.0" />
-	<property name="mass" value="0.1" /> <!-- in kg-->
-	<property name="ixx_com_cs" value="0.01" /> <!-- at center of mass aligned with coordinate system, kg*m^2-->
-	<property name="ixy_com_cs" value="0.0" /> <!-- at center of mass aligned with coordinate system, kg*m^2-->
-	<property name="ixz_com_cs" value="0.0" /> <!-- at center of mass aligned with coordinate system, kg*m^2-->
-	<property name="iyy_com_cs" value="0.01" /> <!-- at center of mass aligned with coordinate system, kg*m^2-->
-	<property name="iyz_com_cs" value="0.00" /> <!-- at center of mass aligned with coordinate system, kg*m^2-->
-	<property name="izz_com_cs" value="0.01" /> <!-- at center of mass aligned with coordinate system, kg*m^2-->
+	<xacro:property name="x_com" value="0.00000000" /> <!-- com : center of mass -->
+	<xacro:property name="y_com" value="0.00000000" /> <!-- com : center of mass -->
+	<xacro:property name="z_com" value="0.00000000" /> <!-- com : center of mass -->
+	<xacro:property name="x_size" value="1.0" />
+	<xacro:property name="y_size" value="1.0" />
+	<xacro:property name="z_size" value="1.0" />
+	<xacro:property name="mass" value="0.1" /> <!-- in kg-->
+	<xacro:property name="ixx_com_cs" value="0.01" /> <!-- at center of mass aligned with coordinate system, kg*m^2-->
+	<xacro:property name="ixy_com_cs" value="0.0" /> <!-- at center of mass aligned with coordinate system, kg*m^2-->
+	<xacro:property name="ixz_com_cs" value="0.0" /> <!-- at center of mass aligned with coordinate system, kg*m^2-->
+	<xacro:property name="iyy_com_cs" value="0.01" /> <!-- at center of mass aligned with coordinate system, kg*m^2-->
+	<xacro:property name="iyz_com_cs" value="0.00" /> <!-- at center of mass aligned with coordinate system, kg*m^2-->
+	<xacro:property name="izz_com_cs" value="0.01" /> <!-- at center of mass aligned with coordinate system, kg*m^2-->
 	<xacro:macro name="kingfisher_part" params="parent name mesh translateX translateY translateZ rotateX rotateY rotateZ color">
 		<joint name="${parent}_${name}_joint" type="fixed">

File: kingfisher_description/urdf/standard.urdf.xacro (robot description, xacro)
@@ -13,6 +13,8 @@
             <bodyName>base_link</bodyName>
             <topicName>imu/data</topicName>
-            <rpyOffsets>0 0 0</rpyOffsets> <!-- deprecated -->
-            <gaussianNoise>0</gaussianNoise> <!-- deprecated -->
+            <rpyOffsets>0 0 0</rpyOffsets>
+            <!-- deprecated -->
+            <gaussianNoise>0</gaussianNoise>
+            <!-- deprecated -->
             <accelDrift>0.5 0.5 0.5</accelDrift>
             <accelGaussianNoise>0.35 0.35 0.3</accelGaussianNoise>
@@ -25,5 +27,5 @@
     <!-- Set up gps configuration -->
     <gazebo>
-        <plugin name="kingfisher_gps" filename="libkingfisher_ros_gps.so">
+        <plugin name="kingfisher_gps" filename="libhector_gazebo_ros_gps.so">
             <alwaysOn>true</alwaysOn>
             <updateRate>10.0</updateRate>
@@ -37,60 +39,8 @@
         </plugin>
     </gazebo>
-    <!-- Set up camera linkage and configuration -->
-    <joint name="base_link_camera_link_joint" type="fixed">
-		<origin xyz="0 0 0.2" rpy="0 0 0" />
-        <parent link="base_link"/>
-        <child link="camera_link" />
-    </joint>
-    <link name="camera_link">
-        <inertial>
-            <mass value="1"/>
-            <origin xyz="0 0 0"/>
-            <inertia ixx="0.1" ixy="0.0" ixz="0.0" iyy="0.1" iyz="0.0" izz="0.1"/>
-        </inertial>
-    </link>
-    <gazebo reference="camera_link">
-        <sensor type="camera" name="camera">
-            <update_rate>30.0</update_rate>
-            <camera name="kingfisher_camera">
-                <horizontal_fov>1.3962634</horizontal_fov>
-                <image>
-                    <width>640</width>
-                    <height>480</height>
-                    <format>R8G8B8</format>
-                </image>
-                <clip>
-                    <near>0.02</near>
-                    <far>300</far>
-                </clip>
-                <noise>
-                    <type>gaussian</type>
-                    <!-- Noise is sampled independently per pixel on each frame.
-                       That pixel's noise value is added to each of its color
-                       channels, which at that point lie in the range [0,1]. -->
-                    <mean>0.0</mean>
-                    <stddev>0.007</stddev>
-                </noise>
-            </camera>
-            <plugin name="camera_controller" filename="libgazebo_ros_camera.so">
-                <alwaysOn>true</alwaysOn>
-                <updateRate>30.0</updateRate>
-                <cameraName>kingfisher/camera</cameraName>
-                <imageTopicName>image_raw</imageTopicName>
-                <cameraInfoTopicName>camera_info</cameraInfoTopicName>
-                <frameName>camera_link</frameName>
-                <hackBaseline>0.07</hackBaseline>
-                <distortionK1>0.0</distortionK1>
-                <distortionK2>0.0</distortionK2>
-                <distortionK3>0.0</distortionK3>
-                <distortionT1>0.0</distortionT1>
-                <distortionT2>0.0</distortionT2>
-            </plugin>
-        </sensor>
-    </gazebo>
     <xacro:if value="$(arg sonar_enabled)">
         <!-- Set up sonar linkage and configuration -->
         <joint name="base_link_sonar_link_joint" type="fixed">
-        <origin xyz="0 0 -0.2" rpy="0 1.57 0" />
+            <origin xyz="0 0 -0.2" rpy="0 1.57 0" />
             <parent link="base_link"/>
             <child link="sonar_link" />
@@ -132,5 +82,5 @@
                     </noise>
                 </ray>
-                <plugin name="kingfisher_ros_sonar_controller" filename="libkingfisher_ros_sonar.so">
+                <plugin name="kingfisher_ros_sonar_controller" filename="libhector_gazebo_ros_sonar.so">
                     <gaussianNoise>0.005</gaussianNoise>
                     <topicName>sonar</topicName>

Commit message: fixed wrong origin for kingfisher base_footprint

File: kingfisher_description/urdf/base.urdf.xacro (robot description, xacro)
@@ -56,5 +56,5 @@
             <origin xyz="0 0 0" rpy="0 0 0" />
             <geometry>
-                <box size="0.001 0.001 0.001" />
+                <box size="1 1 0.001" />
             </geometry>
         </visual>
@@ -64,5 +64,5 @@
     </gazebo>
     <joint name="base_footprint_joint" type="fixed">
-        <origin xyz="0 0 0" rpy="0 0 0" />
+        <origin xyz="0 0 0.2" rpy="0 0 0" />
         <parent link="base_footprint"/>
         <child link="base_link" />
@@ -128,5 +128,5 @@
     <!-- PANEL-LINKS -->
     <!-- Top Plate -->
-    <kingfisher_part parent="base_footprint" name="left_panel" mesh="left_panel" translateX="0.0" translateY="-0.35" translateZ="0.05" rotateX="${M_PI/2}" rotateY="0.0" rotateZ="${M_PI/2}" color="Yellow" />
+    <!-- <kingfisher_part parent="base_footprint" name="left_panel" mesh="left_panel" translateX="0.0" translateY="-0.35" translateZ="0.05" rotateX="${M_PI/2}" rotateY="0.0" rotateZ="${M_PI/2}" color="Yellow" />
     <gazebo reference="base_footprint_left_panel_part">
         <material>Gazebo/Yellow</material>
@@ -135,5 +135,5 @@
     <gazebo reference="base_footprint_right_panel_part">
         <material>Gazebo/Yellow</material>
-    </gazebo>
+    </gazebo> -->
     <!--Gazebo Plugin for simulating Kingfisher dynamics-->
     <!-- <gazebo><plugin name="kingfisher_dynamic" filename="libkingfisher_gazebo_plugins.so"><maxForce>62.0</maxForce><bodyName>base_link</bodyName><waterDensity>997.7735</waterDensity><waterLevel>5</waterLevel><xyzDampingFactor>20.0</xyzDampingFactor><yawDampingFactor>20.0</yawDampingFactor><rolPitDampingFactor>5.0</rolPitDampingFactor></plugin></gazebo> -->

File: kingfisher_description/urdf/kingfisher_robotx.xacro (robot description, xacro)
@@ -26,3 +26,6 @@
   <xacro:include filename="$(find kingfisher_description)/urdf/sensor_p3d.xacro" />
   <xacro:kingfisher_gazebo_p3d name="kingfisher_p3d"/>
+  <!-- Attach Sonar plugin -->
+  <xacro:include filename="$(find kingfisher_description)/urdf/sensor_sonar.xacro" />
+  <xacro:kingfisher_gazebo_p3d name="kingfisher_sonar"/>
 </robot>

File: kingfisher_description/urdf/sensor_gps.xacro (robot description, xacro)
@@ -24,2 +24,16 @@
     </xacro:macro>
 </robot>
+<!-- Reference gps configuration -->
+<!-- <gazebo>
+    <plugin name="kingfisher_gps" filename="libhector_gazebo_ros_gps.so">
+        <alwaysOn>true</alwaysOn>
+        <updateRate>10.0</updateRate>
+        <bodyName>base_link</bodyName>
+        <topicName>navsat/fix</topicName>
+        <velocityTopicName>navsat/vel</velocityTopicName>
+        <drift>5.0 5.0 5.0</drift>
+        <gaussianNoise>0.1 0.1 0.1</gaussianNoise>
+        <velocityDrift>0 0 0</velocityDrift>
+        <velocityGaussianNoise>0.1 0.1 0.1</velocityGaussianNoise>
+    </plugin>
+</gazebo> -->

File: kingfisher_description/urdf/sensor_imu.xacro (robot description, xacro)
@@ -29,2 +29,18 @@
     </xacro:macro>
 </robot>
+    <!-- Reference Setup imu configuration -->
+    <!-- <gazebo>
+        <plugin name="kingfisher_imu" filename="libgazebo_ros_imu.so">
+            <updateRate>20.0</updateRate>
+            <bodyName>base_link</bodyName>
+            <topicName>imu/data</topicName>
+            <rpyOffsets>0 0 0</rpyOffsets>
+            <gaussianNoise>0</gaussianNoise>
+            <accelDrift>0.5 0.5 0.5</accelDrift>
+            <accelGaussianNoise>0.35 0.35 0.3</accelGaussianNoise>
+            <rateDrift>0.1 0.1 0.1</rateDrift>
+            <rateGaussianNoise>0.05 0.05 0.015</rateGaussianNoise>
+            <headingDrift>0.1</headingDrift>
+            <headingGaussianNoise>0.05</headingGaussianNoise>
+        </plugin>
+    </gazebo> -->

File: kingfisher_description/urdf/standard.urdf.xacro (robot description, xacro)
@@ -7,36 +7,4 @@
     <!-- Included URDF Files -->
     <xacro:include filename="$(find kingfisher_description)/urdf/base.urdf.xacro" />
-    <!-- Set up imu configuration -->
-    <gazebo>
-        <plugin name="kingfisher_imu" filename="libgazebo_ros_imu.so">
-            <updateRate>20.0</updateRate>
-            <bodyName>base_link</bodyName>
-            <topicName>imu/data</topicName>
-            <rpyOffsets>0 0 0</rpyOffsets>
-            <!-- deprecated -->
-            <gaussianNoise>0</gaussianNoise>
-            <!-- deprecated -->
-            <accelDrift>0.5 0.5 0.5</accelDrift>
-            <accelGaussianNoise>0.35 0.35 0.3</accelGaussianNoise>
-            <rateDrift>0.1 0.1 0.1</rateDrift>
-            <rateGaussianNoise>0.05 0.05 0.015</rateGaussianNoise>
-            <headingDrift>0.1</headingDrift>
-            <headingGaussianNoise>0.05</headingGaussianNoise>
-        </plugin>
-    </gazebo>
-    <!-- Set up gps configuration -->
-    <gazebo>
-        <plugin name="kingfisher_gps" filename="libhector_gazebo_ros_gps.so">
-            <alwaysOn>true</alwaysOn>
-            <updateRate>10.0</updateRate>
-            <bodyName>base_link</bodyName>
-            <topicName>navsat/fix</topicName>
-            <velocityTopicName>navsat/vel</velocityTopicName>
-            <drift>5.0 5.0 5.0</drift>
-            <gaussianNoise>0.1 0.1 0.1</gaussianNoise>
-            <velocityDrift>0 0 0</velocityDrift>
-            <velocityGaussianNoise>0.1 0.1 0.1</velocityGaussianNoise>
-        </plugin>
-    </gazebo>
     <xacro:if value="$(arg sonar_enabled)">
         <!-- Set up sonar linkage and configuration -->
@@ -53,43 +21,4 @@
             </inertial>
         </link>
-        <gazebo reference="sonar_link">
-            <sensor type="ray" name="sonar_sensor">
-                <pose>0 0 0 0 0 0</pose>
-                <visualize>false</visualize>
-                <update_rate>20</update_rate>
-                <ray>
-                    <scan>
-                        <horizontal>
-                            <samples>3</samples>
-                            <resolution>1</resolution>
-                            <min_angle>${-5*M_PI/180}</min_angle>
-                            <max_angle>${5*M_PI/180}</max_angle>
-                        </horizontal>
-                    </scan>
-                    <range>
-                        <min>0.10</min>
-                        <max>30.0</max>
-                        <resolution>0.01</resolution>
-                    </range>
-                    <noise>
-                        <type>gaussian</type>
-                        <!-- Noise parameters based on published spec for Hokuyo laser
-                             achieving "+-30mm" accuracy at range < 10m.  A mean of 0.0m and
-                             stddev of 0.01m will put 99.7% of samples within 0.03m of the true
-                             reading. -->
-                        <mean>0.0</mean>
-                        <stddev>0.01</stddev>
-                    </noise>
-                </ray>
-                <plugin name="kingfisher_ros_sonar_controller" filename="libhector_gazebo_ros_sonar.so">
-                    <gaussianNoise>0.005</gaussianNoise>
-                    <topicName>sonar</topicName>
-                    <frameId>sonar_link</frameId>
-                    <offset>0</offset>
-                    <drift>0</drift>
-                    <driftFrequency>0</driftFrequency>
-                </plugin>
-            </sensor>
-        </gazebo>
     </xacro:if>
 </robot>
