Commit message: corrections on kingfisher URDF

File: kingfisher_description/urdf/base.urdf.xacro (robot description, xacro)
@@ -53,10 +53,5 @@
             <inertia ixx="0.0001" ixy="0.0" ixz="0.0" iyy="0.0001" iyz="0.0" izz="0.0001" />
         </inertial>
-        <visual>
-            <origin xyz="0 0 0" rpy="0 0 0" />
-            <geometry>
-                <box size="1 1 0.001" />
-            </geometry>
-        </visual>
+        <!-- <visual><origin xyz="0 0 0" rpy="0 0 0" /><geometry><box size="1 1 0.001" /></geometry></visual> -->
     </link>
     <gazebo reference="base_footprint">
@@ -92,4 +87,7 @@
             </geometry>
         </collision>
+        <gazebo reference="base_link">
+            <material>Gazebo/Orange</material>
+        </gazebo>
     </link>
     <xacro:property name="camera_link" value="0.05" />
@@ -128,12 +126,5 @@
     <!-- PANEL-LINKS -->
     <!-- Top Plate -->
-    <!-- <kingfisher_part parent="base_footprint" name="left_panel" mesh="left_panel" translateX="0.0" translateY="-0.35" translateZ="0.05" rotateX="${M_PI/2}" rotateY="0.0" rotateZ="${M_PI/2}" color="Yellow" />
-    <gazebo reference="base_footprint_left_panel_part">
-        <material>Gazebo/Yellow</material>
-    </gazebo>
-    <kingfisher_part parent="base_footprint" name="right_panel" mesh="right_panel" translateX="0.0" translateY="0.35" translateZ="0.05" rotateX="${M_PI/2}" rotateY="0.0" rotateZ="${-M_PI/2}" color="Yellow" />
-    <gazebo reference="base_footprint_right_panel_part">
-        <material>Gazebo/Yellow</material>
-    </gazebo> -->
+    <!-- <kingfisher_part parent="base_footprint" name="left_panel" mesh="left_panel" translateX="0.0" translateY="-0.35" translateZ="0.05" rotateX="${M_PI/2}" rotateY="0.0" rotateZ="${M_PI/2}" color="Yellow" /><gazebo reference="base_footprint_left_panel_part"><material>Gazebo/Yellow</material></gazebo><kingfisher_part parent="base_footprint" name="right_panel" mesh="right_panel" translateX="0.0" translateY="0.35" translateZ="0.05" rotateX="${M_PI/2}" rotateY="0.0" rotateZ="${-M_PI/2}" color="Yellow" /><gazebo reference="base_footprint_right_panel_part"><material>Gazebo/Yellow</material></gazebo> -->
     <!--Gazebo Plugin for simulating Kingfisher dynamics-->
     <!-- <gazebo><plugin name="kingfisher_dynamic" filename="libkingfisher_gazebo_plugins.so"><maxForce>62.0</maxForce><bodyName>base_link</bodyName><waterDensity>997.7735</waterDensity><waterLevel>5</waterLevel><xyzDampingFactor>20.0</xyzDampingFactor><yawDampingFactor>20.0</yawDampingFactor><rolPitDampingFactor>5.0</rolPitDampingFactor></plugin></gazebo> -->

Commit message: proper collision box for kf

File: kingfisher_description/urdf/base.urdf.xacro (robot description, xacro)
@@ -78,22 +78,20 @@
                 <mesh filename="package://kingfisher_description/meshes/kingfisher_base.stl" />
             </geometry>
-            <material name="DarkGray" />
+            <!-- <material name="DarkGray" /> -->
+            <material name="Yellow" />
         </visual>
         <collision>
-            <origin xyz="0 0 0" rpy="0 0 0" />
+            <origin xyz="0.02 0 -0.05" rpy="0 0 0" />
             <geometry>
-                <box size = "0.1 0.1 0.1"/>
+                <box size = "1.35 0.98 0.32"/>
                 <!--making it slightly bigger in x and z direction-->
             </geometry>
         </collision>
-        <gazebo reference="base_link">
-            <material>Gazebo/Orange</material>
-        </gazebo>
     </link>
     <xacro:property name="camera_link" value="0.05" />
     <!-- Size of square 'camera' box -->
-    <joint name="camera_joint" type="fixed">
+    <joint name="camera_joint" type="continuous">
         <axis xyz="0 1 0" />
-        <origin xyz="${camera_link} 0 1" rpy="0 0 0"/>
+        <origin xyz="0.3 0 0.07" rpy="0 0 0"/>
         <parent link="base_link"/>
         <child link="camera_link"/>
@@ -121,5 +119,5 @@
     </link>
     <gazebo reference="base_link">
-        <material>Gazebo/FlatBlack</material>
+        <material>Gazebo/Orange</material>
         <turnGravityOff>false</turnGravityOff>
     </gazebo>

Commit message: updated cam position + velodyne

File: kingfisher_description/urdf/base.urdf.xacro (robot description, xacro)
@@ -91,7 +91,7 @@
     <xacro:property name="camera_link" value="0.05" />
     <!-- Size of square 'camera' box -->
-    <joint name="camera_joint" type="continuous">
-        <axis xyz="0 1 0" />
-        <origin xyz="0.3 0 0.07" rpy="0 0 0"/>
+    <joint name="camera_joint" type="fixed">
+        <!-- <axis xyz="0 1 0" /> -->
+        <origin xyz="0.3 0 0.11" rpy="0 0 0"/>
         <parent link="base_link"/>
         <child link="camera_link"/>
@@ -110,5 +110,5 @@
                 <box size="${camera_link} ${camera_link} ${camera_link}"/>
             </geometry>
-            <material name="red"/>
+            <material name="Red"/>
         </visual>
         <inertial>

File: kingfisher_description/urdf/kingfisher_robotx.xacro (robot description, xacro)
@@ -29,3 +29,6 @@
   <xacro:include filename="$(find kingfisher_description)/urdf/sensor_sonar.xacro" />
   <xacro:kingfisher_gazebo_p3d name="kingfisher_sonar"/>
+  <!-- Attach Velodyne plugin -->
+  <xacro:include filename="$(find kingfisher_description)/urdf/sensor_velodyne.xacro" />
+  <xacro:kingfisher_gazebo_velodyne name="kingfisher_velodyne"/>
 </robot>

File: kingfisher_description/urdf/materials.urdf.xacro (robot description, xacro)
@@ -41,3 +41,6 @@
 		<color rgba="0.8 0.8 0.0 1.0"/>
 	</material>
+	<material name="Red">
+		<color rgba="0.8 0.1 0.0 1.0"/>
+	</material>
 </robot>

Commit message: a bit more doc

File: kingfisher_description/urdf/base.urdf.xacro (robot description, xacro)
@@ -102,5 +102,5 @@
             <origin xyz="0 0 0" rpy="0 0 0"/>
             <geometry>
-                <box size="${camera_link} ${camera_link} ${camera_link}"/>
+                <box size="${camera_link} ${camera_link} ${camera_link}"/>fi
             </geometry>
         </collision>

Commit message: July Update

File: kingfisher_description/urdf/base.urdf.xacro (robot description, xacro)
@@ -74,10 +74,10 @@
             <mass value="29" />
             <!--This is the pose of the inertial reference frame, relative to the link reference frame. The origin of the inertial reference frame needs to be at the center of gravity. The axes of the inertial reference frame do not need to be aligned with the principal axes of the inertia.-->
-            <origin xyz="0 0 0" />
+            <origin xyz="0 0 0.18" />
             <!--The 3x3 rotational inertia matrix. Because the rotational inertia matrix is symmetric, only 6 above-diagonal elements of this matrix are specified here, using the attributes ixx, ixy, ixz, iyy, iyz, izz.-->
             <inertia ixx="10" ixy="0" ixz="0" iyy="10" iyz="0" izz="10" />
         </inertial>
         <visual>
-            <origin xyz="0 0 0" rpy="${M_PI/2} 0 ${M_PI/2}" />
+            <origin xyz="0 0 0.18" rpy="${M_PI/2} 0 ${M_PI/2}" />
             <geometry>
                 <mesh filename="package://kingfisher_description/meshes/kingfisher_base.stl" />
@@ -86,5 +86,5 @@
         </visual>
         <collision>
-            <origin xyz="0 0 0" rpy="0 0 0" />
+            <origin xyz="0 0 0.18" rpy="0 0 0" />
             <geometry>
                 <box size = "0.1 0.1 0.1"/>

File: robotx_gazebo/urdf/kingfisher_gazebo_dynamics_plugin.xacro (robot description, xacro)
@@ -34,11 +34,11 @@
 				<!-- Waves x3 -->
 				<wave_n>3</wave_n>
-				<wave_amp0>0.06</wave_amp0>
+				<wave_amp0>0</wave_amp0>
 				<wave_period0>12.6</wave_period0>
 				<wave_direction0>-1 0</wave_direction0>
-				<wave_amp1>0.04</wave_amp1>
+				<wave_amp1>0</wave_amp1>
 				<wave_period1>3.7</wave_period1>
 				<wave_direction1>-0.7 0.7</wave_direction1>
-				<wave_amp2>0.03</wave_amp2>
+				<wave_amp2>0</wave_amp2>
 				<wave_period2>6.3</wave_period2>
 				<wave_direction2>0.7 0.7</wave_direction2>

File: robotx_gazebo/urdf/kingfisher_gazebo_thrust_plugin.xacro (robot description, xacro)
@@ -12,11 +12,11 @@
 				<!-- General dimensions -->
 				<boatArea>0.48</boatArea>
-				<boatWidth>0.98</boatWidth>
-				<boatLength>1.35</boatLength>
+				<boatWidth>4</boatWidth>
+				<boatLength>1</boatLength>
 				<thrustOffsetZ>-0.04</thrustOffsetZ>
 				<!-- Thrust specification -->
 				<maxCmd>1.0</maxCmd>
-				<maxForceFwd>21</maxForceFwd>
-				<maxForceRev>-6</maxForceRev>
+				<maxForceFwd>100</maxForceFwd>
+				<maxForceRev>-50</maxForceRev>
 				<cmdTimeout>1.0</cmdTimeout>
 			</plugin>
