Commit message: wamv description - added sensors

File: wamv_description/urdf/wamv_base.xacro (robot description, xacro)
@@ -1,4 +1,5 @@
 <?xml version="1.0"?>
-<robot xmlns:xacro="http://ros.org/wiki/xacro" name="wam-v">
+<robot
+  xmlns:xacro="http://ros.org/wiki/xacro" name="wam-v">
   <xacro:include filename="properties.urdf.xacro"/>
   <link name="base_link">
@@ -209,5 +210,6 @@
     </collision>
     <inertial>
-      <mass value="180.0"/> <!-- From von Ellenrieder, consistent with WAM-V specs-->
+      <mass value="180.0"/>
+      <!-- From von Ellenrieder, consistent with WAM-V specs-->
       <!--<inertia ixx="200.0" ixy="0.03" ixz="3.09" iyy="500" iyz="-0.05" izz="250.0"/>-->
       <inertia ixx="120.0" ixy="0.0" ixz="0.0" iyy="393" iyz="0.0" izz="446.0"/>

File: wamv_description/urdf/wamv_robotx.xacro (robot description, xacro)
@@ -13,3 +13,15 @@
   <xacro:include filename="$(find robotx_gazebo)/urdf/wamv_gazebo_thrust_plugin.xacro" />
   <xacro:usv_thrust_gazebo name="wamv_thrust_plugin"/>
+    <!-- Attach Camera plugin -->
+  <xacro:include filename="$(find wamv_description)/urdf/sensor_camera.xacro" />
+  <xacro:wamv_gazebo_camera name="wamv_camera1"/>
+  <!-- Attach IMU plugin -->
+  <xacro:include filename="$(find wamv_description)/urdf/sensor_imu.xacro" />
+  <xacro:wamv_gazebo_imu name="wamv_imu"/>
+  <!-- Attach GPS plugin -->
+  <xacro:include filename="$(find wamv_description)/urdf/sensor_gps.xacro" />
+  <xacro:wamv_gazebo_gps name="wamv_gps"/>
+  <!-- Attach P3D plugin -->
+  <xacro:include filename="$(find wamv_description)/urdf/sensor_p3d.xacro" />
+  <xacro:wamv_gazebo_p3d name="wamv_p3d"/>
 </robot>

Commit message: Added task worlds

File: wamv_description/urdf/wamv_base.xacro (robot description, xacro)
@@ -224,5 +224,5 @@
   <link name="front_camera_link"/>
   <joint name="front_camera_joint" type="fixed">
-    <origin xyz="0.5 0 1.5"/>
+    <origin xyz="0.8 0 1.5"/>
     <parent link="base_link"/>
     <child link="front_camera_link"/>
